File: OverVoltageProtection.kicad_sch (KiCad schematic)
At the start: 18 parts, among them Q3 IRFR210PBF, Q4 IRFR210PBF, U1 LM74800QDRRRQ1, U2 LM5069MM-2_NOPB

Commit message: sample layout
Parts:
- added C1: 1uF, symbol PCM_Elektuur:C
- added C7: 150nF, symbol PCM_Elektuur:C
- added C8: 330uF, symbol PCM_Elektuur:C
- added D5: SMBJ30A-13-F, SMBJ30A-13-F:DIOM5336X250N, symbol SMBJ30A-13-F:SMBJ30A-13-F
- added D6: SS310, Diode_SMD:D_SMA, symbol Diode:SS310
- added Q1: IRFR210PBF, Package_TO_SOT_SMD:TO-252-3_TabPin2, symbol Device:Q_NMOS_Depletion_GDS
- added R1, R4: 47.5k, symbol PCM_Elektuur:R
- added R10: 100k, symbol PCM_Elektuur:R
- added R2: 8.25k, symbol PCM_Elektuur:R
- added R7: 4.22k, symbol PCM_Elektuur:R
- added R8: 0.004R, symbol PCM_Elektuur:R
- added R9: 15.8k, symbol PCM_Elektuur:R
Connections:
- net OUT is gone; now on net V_FILTERED: C6.1 (+), D4.2 (A), Q3.3 (S), Q4.3 (S), U1.2 (A), U1.9 (OUT)
- net GND: now also U2.5 (GND), C1.2 (-), C7.2 (-), C8.2 (-), D5.2, D6.2 (A), R2.2 (-), R7.2 (-), R9.2 (-)
- net VOUT: now also U2.2 (VIN), C1.1 (+), D5.1, R1.1 (+), R4.1 (+), R8.1 (+)
- net SENSE: now reaches U2.1 (SENSE)
- net SENSE: now also Q1.2 (D), R8.2 (-)
- net at U2.10 (GATE): now also Q1.1 (G)
- net UVLO: now reaches U2.3 (UVLO)
- net UVLO: now also R1.2 (-), R2.1 (+)
- net at U2.4 (OVLO): now also R4.2 (-), R7.1 (+)
- net at U2.6 (TIMER): now also C7.1 (+)
- net at U2.7 (PWR): now also R9.1 (+)
- net PGOOD: now reaches U2.8 (PGD)
- net PGOOD: now also R10.2 (-)
- net V_FILTERED: now reaches U2.9 (OUT)
- net V_FILTERED: now also C8.1 (+), D6.1 (K), Q1.3 (S)
- new net +5V: R10.1 (+)
Other:
- moved on the sheet: C2, C3, C4, C5, C6, D1, D2, D3, D4, JP1, JP2, Q3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

Commit message: prototyple schematics finished
Parts:
- removed C1, C6: 1uF, symbol PCM_Elektuur:C
- removed C7: 150nF, symbol PCM_Elektuur:C
- removed C8: 330uF, symbol PCM_Elektuur:C
- removed D5: SMBJ30A-13-F, SMBJ30A-13-F:DIOM5336X250N, symbol SMBJ30A-13-F:SMBJ30A-13-F
- removed D6: SS310, Diode_SMD:D_SMA, symbol Diode:SS310
- removed JP1, JP2: Jumper_2_Open, symbol Jumper:Jumper_2_Open
- removed Q1, Q3: IRFR210PBF, Package_TO_SOT_SMD:TO-252-3_TabPin2, symbol Device:Q_NMOS_Depletion_GDS
- removed R1, R4: 47.5k, symbol PCM_Elektuur:R
- removed R10: 100k, symbol PCM_Elektuur:R
- removed R2: 8.25k, symbol PCM_Elektuur:R
- removed R7: 4.22k, symbol PCM_Elektuur:R
- removed R8: 0.004R, symbol PCM_Elektuur:R
- removed R9: 15.8k, symbol PCM_Elektuur:R
- removed U2: LM5069MM-2_NOPB, LM5069MM-2_NOPB:SOP50P490X110-10N, symbol LM5069MM-2_NOPB:LM5069MM-2_NOPB
- added C10, C9: 0.1uF, symbol PCM_Elektuur:C
- added C11: 1uF, symbol PCM_Elektuur:C
- added C12: 0.01uF, symbol PCM_Elektuur:C
- added C13, C16, C17: 100nF, symbol PCM_Elektuur:C
- added C14: 0.56uF, symbol PCM_Elektuur:C
- added C15: 1000pF, symbol PCM_Elektuur:C
- added C18: 100uF, symbol PCM_Elektuur:C
- added D7: 1N6263, Diode_THT:D_DO-35_SOD27_P7.62mm_Horizontal, symbol Diode:1N6263
- added Q2, Q3: SQJQ466E, Package_TO_SOT_SMD:LFPAK88, symbol Transistor_FET:SQJQ466E
- added R1, R16: R-nonlin, symbol PCM_Elektuur:R-nonlin
- added R11: 100R, symbol PCM_Elektuur:R
- added R12: 95.3k, symbol PCM_Elektuur:R
- added R13: 13.7k, symbol PCM_Elektuur:R
- added R14: 54.9k, symbol PCM_Elektuur:R
- added R15: 0.004R, symbol PCM_Elektuur:R
- added U3: LM5069MM-2_NOPB, LM5069MM-2_NOPB:SOP50P490X110-10N, symbol LM5069MM-2_NOPB:LM5069MM-2_NOPB
- C2: value 0.1uF -> 47uF
- C5: value 47uF -> 2.2uF
Connections:
- net DGATE: now also Q2.1 (G)
- net GND: now also C10.2 (-), C11.2 (-), C13.2 (-), C17.2 (-), C18.2 (-), C9.2 (-), R1.1 (+), R16.1 (+); no longer C3.2 (-), D3.2 (A), R6.2 (-), U1.7 (GND)
- net HGATE: now also R11.1 (+)
- net SENSE: now also Q3.2 (S), Q3.3 (S), Q3.4 (S), R15.2 (-), U3.1 (SENSE)
- net UVLO: now also R12.2 (-), R13.1 (+), U3.3 (UVLO)
- net VBat: now also C10.1 (+), C9.1 (+); no longer C2.1 (+)
- net VOUT: now also C2.1 (+), R5.1 (+), C13.1 (+), C15.1 (+), Q2.5 (D), R12.1 (+), R15.1 (+), U3.2 (VIN)
- net V_FILTERED: now also C16.1 (+), C17.1 (+), C18.1 (+), Q3.5 (D); no longer D4.2 (A), Q4.3 (S), U1.2 (A), U1.9 (OUT)
- net at D1.2 (A2), D2.2 (A2): now also C11.1 (+)
- net OV: no longer names the net of R5.2 (-), R6.1 (+), U1.5 (OV)
- new net: C12.1 (+), R11.2 (-)
- new net: R14.1 (+), U3.7 (PWR)
- new net: D7.1 (K), Q3.1 (G), U3.10 (GATE)
- new net: C14.1 (+), U3.6 (TIMER)
- new net GNDA: C12.2 (-), C14.2 (-), C15.2 (-), C16.2 (-), C3.2 (-), D3.2 (A), D7.2 (A), R1.2 (-), R13.2 (-), R14.2 (-), R16.2 (-), R6.2 (-), U1.7 (GND), U3.4 (OVLO), U3.5 (GND)
- new net OUT: D4.2 (A), Q2.2 (S), Q2.3 (S), Q2.4 (S), Q4.3 (S), U1.2 (A), U1.9 (OUT)
Other:
- moved on the sheet: C3, C4, C5, D1, D2, D3, D4, Q4, R3, R5, R6, U1

Commit message: completed schematics
Parts:
- removed R1, R16: R-nonlin, symbol PCM_Elektuur:R-nonlin
- added D5: BAV20WS-TP, Diode_SMD:D_SOD-323, symbol Device:D
- added JP1: Jumper_2_Bridged, Jumper:SolderJumper-2_P1.3mm_Bridged_RoundedPad1.0x1.5mm, symbol Jumper:Jumper_2_Bridged
- C10, C4, C9: value 0.1uF -> 100nF; footprint (none) -> Capacitor_SMD:C_0805_2012Metric
- C11, C14, C3: footprint (none) -> Capacitor_SMD:C_1206_3216Metric
- C12: value 0.01uF -> 10nF; footprint (none) -> Capacitor_SMD:C_0805_2012Metric
- C13, C16, C5: footprint (none) -> Capacitor_SMD:C_0805_2012Metric
- C15: footprint (none) -> Capacitor_SMD:C_0603_1608Metric
- C17: value 100nF -> 100uF; footprint (none) -> Capacitor_SMD:CP_Elec_8x10
- C18, C2: footprint (none) -> Capacitor_SMD:CP_Elec_8x10
- D1: value SMAJ250A -> 5.0SMDJ120A; footprint Diode_SMD:D_SMA -> Diode_SMD:D_SMC
- D2: value SMAJ250CA -> 5.0SMDJ33CA; footprint Diode_SMD:D_SMA -> Diode_SMD:D_SMC
- R11, R12, R13, R14, R3, R5, R6: footprint (none) -> Resistor_SMD:R_1206_3216Metric_Pad1.30x1.75mm_HandSolder
- R15: footprint (none) -> Resistor_SMD:R_Shunt_Vishay_WSR2_WSR3_KelvinConnection
Connections:
- net VOUT is gone; now on net V_FILTERED: C13.1 (+), C15.1 (+), C2.1 (+), C5.1 (+), Q2.5 (D), R12.1 (+), R15.1 (+), R5.1 (+), U1.12 (C), U3.2 (VIN)
- net GND: now also C12.2 (-), C14.2 (-), C16.2 (-), C3.2 (-), D3.2 (A), D7.2 (A), R13.2 (-), R14.2 (-), R6.2 (-), U1.7 (GND), U3.4 (OVLO), U3.5 (GND), D5.1 (K), D5.2 (A)
- net GNDA: no longer C12.2 (-), C14.2 (-), C16.2 (-), C3.2 (-), D3.2 (A), D7.2 (A), R13.2 (-), R14.2 (-), R6.2 (-), U1.7 (GND), U3.4 (OVLO), U3.5 (GND)
- net VS: now also JP1.2 (B); no longer U1.6 (EN/UVLO)
- net V_FILTERED: now also U3.9 (OUT)
- new net: JP1.1 (A), U1.6 (EN/UVLO)
- no-connect marks 1 -> 2
Other:
- moved on the sheet: C12, C15, C16, C17, C18, D7, R11

Commit message: finished layout
Parts:
- removed D5: BAV20WS-TP, Diode_SMD:D_SOD-323, symbol Device:D
- removed JP1: Jumper_2_Bridged, Jumper:SolderJumper-2_P1.3mm_Bridged_RoundedPad1.0x1.5mm, symbol Jumper:Jumper_2_Bridged
- added H1, H2, H3, H4: MountingHole_M3_3.2mm_Pad, PCM_SL_Mechanical:MountingHole_3.2mm_Pad, symbol PCM_SL_Mechanical:MountingHole_M3_3.2mm_Pad
Connections:
- net GNDA is gone; now on net GND: C15.2 (-)
- net GND: now also H1.1, H4.1
- net OUT: now also Q2.5 (D); no longer Q2.2 (S), Q2.3 (S), Q2.4 (S)
- net VBat: now also H2.1
- net VS: now also U1.6 (EN/UVLO)
- net V_FILTERED: now also H3.1; no longer C13.1 (+), C15.1 (+), C2.1 (+), C5.1 (+), Q2.5 (D), R12.1 (+), R15.1 (+), U3.2 (VIN)
- new net V_INTER: C13.1 (+), C15.1 (+), C2.1 (+), C5.1 (+), Q2.2 (S), Q2.3 (S), Q2.4 (S), R12.1 (+), R15.1 (+), U3.2 (VIN)
Other:
- moved on the sheet: Q2

Commit message: bug fixing
Parts:
- removed H1, H2, H3, H4: MountingHole_M3_3.2mm_Pad, PCM_SL_Mechanical:MountingHole_3.2mm_Pad, symbol PCM_SL_Mechanical:MountingHole_M3_3.2mm_Pad
- added H1, H6, H7, H8: MountingHole_Pad, MountingHole:MountingHole_3.2mm_M3_Pad, symbol Mechanical:MountingHole_Pad
Connections:
- net GND: now also H1.1, H8.1
- net VBat: now also H6.1
- net V_FILTERED: now also H7.1
Changed lines of the file:
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@@
 	)
 	(symbol
-		(lib_id "PCM_SL_Mechanical:MountingHole_M3_3.2mm_Pad")
-		(at 34.29 88.9 0)
+		(lib_id "Mechanical:MountingHole_Pad")
+		(at 72.39 74.93 0)
 		(unit 1)
-		(exclude_from_sim no)
-		(in_bom yes)
+		(exclude_from_sim yes)
+		(in_bom no)
 		(on_board yes)
 		(dnp no)
 		(fields_autoplaced yes)
-		(property "Reference" "H1"
-			(at 38.1 87.6299 0)
+		(property "Reference" "H7"
+			(at 74.93 72.3899 0)
 			(effects
 				(font
@@
 			)
 		)
-		(property "Value" "MountingHole_M3_3.2mm_Pad"
-			(at 38.1 90.1699 0)
+		(property "Value" "MountingHole_Pad"
+			(at 74.93 74.9299 0)
 			(effects
 				(font
@@
 			)
 		)
-		(property "Footprint" "PCM_SL_Mechanical:MountingHole_3.2mm_Pad"
-			(at 34.29 92.71 0)
+		(property "Footprint" "MountingHole:MountingHole_3.2mm_M3_Pad"
+			(at 72.39 74.93 0)
 			(effects
 				(font
@@
 			)
 		)
-		(property "Datasheet" ""
-			(at 34.29 88.9 0)
+		(property "Datasheet" "~"
+			(at 72.39 74.93 0)
 			(effects
 				(font
@@
 			)
 		)
-		(property "Description" "3.2mm Diameter Mounting Hole Pad (M3)"
-			(at 34.29 88.9 0)
+		(property "Description" "Mounting Hole with connection"
+			(at 72.39 74.93 0)
 			(effects
 				(font
@@
 			(project "OverVoltageProtection"
 				(path "/3ab01156-4af1-4058-a55c-fa6294991d75"
-					(reference "H1")
+					(reference "H7")
 					(unit 1)
 				)
@@
 	)
 	(symbol
-		(lib_id "PCM_SL_Mechanical:MountingHole_M3_3.2mm_Pad")
-		(at 72.39 72.39 0)
-		(unit 1)
-		(exclude_from_sim no)
-		(in_bom yes)
-		(on_board yes)
-		(dnp no)
-		(fields_autoplaced yes)
-		(property "Reference" "H3"
-			(at 76.2 71.1199 0)
-			(effects
-				(font
-					(size 1.27 1.27)
-				)
-				(justify left)
-			)
-		)
-		(property "Value" "MountingHole_M3_3.2mm_Pad"
-			(at 76.2 73.6599 0)
-			(effects
-				(font
-					(size 1.27 1.27)
-				)
-				(justify left)
-			)
-		)
-		(property "Footprint" "PCM_SL_Mechanical:MountingHole_3.2mm_Pad"
-			(at 72.39 76.2 0)
-			(effects
-				(font
-					(size 1.27 1.27)
-				)
-				(hide yes)
-			)
-		)
-		(property "Datasheet" ""
-			(at 72.39 72.39 0)
-			(effects
-				(font
-					(size 1.27 1.27)
-				)
-				(hide yes)
-			)
-		)
-		(property "Description" "3.2mm Diameter Mounting Hole Pad (M3)"
-			(at 72.39 72.39 0)
-			(effects
-				(font
-					(size 1.27 1.27)
-				)
-				(hide yes)
-			)
-		)
-		(pin "1"
-		)
-		(instances
-			(project "OverVoltageProtection"
-				(path "/3ab01156-4af1-4058-a55c-fa6294991d75"
-					(reference "H3")
-					(unit 1)
-				)
-			)
-		)
-	)
-	(symbol
 		(lib_id "power:GND2")
 		(at 115.57 156.21 0)
@@
 	)
 	(symbol
+		(lib_id "Mechanical:MountingHole_Pad")
+		(at 34.29 91.44 0)
+		(unit 1)
+		(exclude_from_sim yes)
+		(in_bom no)
+		(on_board yes)
+		(dnp no)
+		(fields_autoplaced yes)
+		(property "Reference" "H1"
+			(at 36.83 88.8999 0)
+			(effects
+				(font
+					(size 1.27 1.27)
+				)
+				(justify left)
+			)
+		)
+		(property "Value" "MountingHole_Pad"
+			(at 36.83 91.4399 0)
+			(effects
+				(font
+					(size 1.27 1.27)
+				)
+				(justify left)
+			)
+		)
+		(property "Footprint" "MountingHole:MountingHole_3.2mm_M3_Pad"
+			(at 34.29 91.44 0)
+			(effects
+				(font
+					(size 1.27 1.27)
+				)
+				(hide yes)
+			)
+		)
+		(property "Datasheet" "~"
+			(at 34.29 91.44 0)
+			(effects
+				(font
+					(size 1.27 1.27)
+				)
+				(hide yes)
+			)
+		)
+		(property "Description" "Mounting Hole with connection"
+			(at 34.29 91.44 0)
+			(effects
+				(font
+					(size 1.27 1.27)
+				)
+				(hide yes)
+			)
+		)
+		(pin "1"
+		)
+		(instances
+			(project "OverVoltageProtection"
+				(path "/3ab01156-4af1-4058-a55c-fa6294991d75"
+					(reference "H1")
+					(unit 1)
+				)
+			)
+		)
+	)
+	(symbol
 		(lib_id "Transistor_FET:SQJQ466E")
 		(at 149.86 35.56 90)
@@
 	)
 	(symbol
-		(lib_id "PCM_SL_Mechanical:MountingHole_M3_3.2mm_Pad")
-		(at 72.39 88.9 0)
-		(unit 1)
-		(exclude_from_sim no)
-		(in_bom yes)
-		(on_board yes)
-		(dnp no)
-		(fields_autoplaced yes)
-		(property "Reference" "H4"
-			(at 76.2 87.6299 0)
-			(effects
-				(font
-					(size 1.27 1.27)
-				)
-				(justify left)
-			)
-		)
-		(property "Value" "MountingHole_M3_3.2mm_Pad"
-			(at 76.2 90.1699 0)
-			(effects
-				(font
-					(size 1.27 1.27)
-				)
-				(justify left)
-			)
-		)
-		(property "Footprint" "PCM_SL_Mechanical:MountingHole_3.2mm_Pad"
-			(at 72.39 92.71 0)
-			(effects
-				(font
-					(size 1.27 1.27)
-				)
-				(hide yes)
-			)
-		)
-		(property "Datasheet" ""
-			(at 72.39 88.9 0)
-			(effects
-				(font
-					(size 1.27 1.27)
-				)
-				(hide yes)
-			)
-		)
-		(property "Description" "3.2mm Diameter Mounting Hole Pad (M3)"
-			(at 72.39 88.9 0)
-			(effects
-				(font
-					(size 1.27 1.27)
-				)
-				(hide yes)
-			)
-		)
-		(pin "1"
-		)
-		(instances
-			(project "OverVoltageProtection"
-				(path "/3ab01156-4af1-4058-a55c-fa6294991d75"
-					(reference "H4")
-					(unit 1)
-				)
-			)
-		)
-	)
-	(symbol
 		(lib_id "PCM_Elektuur:C")
 		(at 191.77 111.76 0)
@@
 	)
 	(symbol
-		(lib_id "PCM_SL_Mechanical:MountingHole_M3_3.2mm_Pad")
-		(at 34.29 72.39 0)
+		(lib_id "Mechanical:MountingHole_Pad")
+		(at 72.39 91.44 0)
 		(unit 1)
-		(exclude_from_sim no)
-		(in_bom yes)
+		(exclude_from_sim yes)
+		(in_bom no)
 		(on_board yes)
 		(dnp no)
 		(fields_autoplaced yes)
-		(property "Reference" "H2"
-			(at 38.1 71.1199 0)
+		(property "Reference" "H8"
+			(at 74.93 88.8999 0)
 			(effects
 				(font
@@
 			)
 		)
-		(property "Value" "MountingHole_M3_3.2mm_Pad"
-			(at 38.1 73.6599 0)
+		(property "Value" "MountingHole_Pad"
+			(at 74.93 91.4399 0)
 			(effects
 				(font
@@
 			)
 		)
-		(property "Footprint" "PCM_SL_Mechanical:MountingHole_3.2mm_Pad"
-			(at 34.29 76.2 0)
+		(property "Footprint" "MountingHole:MountingHole_3.2mm_M3_Pad"
+			(at 72.39 91.44 0)
 			(effects
 				(font
@@
 			)
 		)
-		(property "Datasheet" ""
-			(at 34.29 72.39 0)
+		(property "Datasheet" "~"
+			(at 72.39 91.44 0)
 			(effects
 				(font
@@
 			)
 		)
-		(property "Description" "3.2mm Diameter Mounting Hole Pad (M3)"
-			(at 34.29 72.39 0)
+		(property "Description" "Mounting Hole with connection"
+			(at 72.39 91.44 0)
 			(effects
 				(font
@@
 		)
 		(instances
-			(project ""
+			(project "OverVoltageProtection"
 				(path "/3ab01156-4af1-4058-a55c-fa6294991d75"
-					(reference "H2")
+					(reference "H8")
 					(unit 1)
 				)
@@
 					(unit 1)
 				)
+			)
+		)
+	)
+	(symbol
+		(lib_id "Mechanical:MountingHole_Pad")
+		(at 34.29 74.93 0)
+		(unit 1)
+		(exclude_from_sim yes)
+		(in_bom no)
+		(on_board yes)
+		(dnp no)
+		(fields_autoplaced yes)
+		(property "Reference" "H6"
+			(at 36.83 72.3899 0)
+			(effects
+				(font
+					(size 1.27 1.27)
+				)
+				(justify left)
+			)
+		)
+		(property "Value" "MountingHole_Pad"
+			(at 36.83 74.9299 0)
+			(effects
+				(font
+					(size 1.27 1.27)
+				)
+				(justify left)
+			)
+		)
+		(property "Footprint" "MountingHole:MountingHole_3.2mm_M3_Pad"
+			(at 34.29 74.93 0)
+			(effects
+				(font
+					(size 1.27 1.27)
+				)
+				(hide yes)
+			)
+		)
+		(property "Datasheet" "~"
+			(at 34.29 74.93 0)
+			(effects
+				(font
+					(size 1.27 1.27)
+				)
+				(hide yes)
+			)
+		)
+		(property "Description" "Mounting Hole with connection"
+			(at 34.29 74.93 0)
+			(effects
+				(font
+					(size 1.27 1.27)
+				)
+				(hide yes)
+			)
+		)
+		(pin "1"
+		)
+		(instances
+			(project "OverVoltageProtection"
+				(path "/3ab01156-4af1-4058-a55c-fa6294991d75"
+					(reference "H6")
+					(unit 1)
+				)

Commit message: Reworked schematics
Parts:
- removed C10, C13, C16, C4, C9: 100nF, Capacitor_SMD:C_0805_2012Metric, symbol PCM_Elektuur:C
- removed C11, C3: 1uF, Capacitor_SMD:C_1206_3216Metric, symbol PCM_Elektuur:C
- removed C12: 10nF, Capacitor_SMD:C_0805_2012Metric, symbol PCM_Elektuur:C
- removed C14: 0.56uF, Capacitor_SMD:C_1206_3216Metric, symbol PCM_Elektuur:C
- removed C15: 1000pF, Capacitor_SMD:C_0603_1608Metric, symbol PCM_Elektuur:C
- removed C17, C18: 100uF, Capacitor_SMD:CP_Elec_8x10, symbol PCM_Elektuur:C
- removed C2: 47uF, Capacitor_SMD:CP_Elec_8x10, symbol PCM_Elektuur:C
- removed C5: 2.2uF, Capacitor_SMD:C_0805_2012Metric, symbol PCM_Elektuur:C
- removed D1: 5.0SMDJ120A, Diode_SMD:D_SMC, symbol Diode:SMAJ250A
- removed D2: 5.0SMDJ33CA, Diode_SMD:D_SMC, symbol Diode:SMAJ250CA
- removed D3, D7: 1N6263, Diode_THT:D_DO-35_SOD27_P7.62mm_Horizontal, symbol Diode:1N6263
- removed D4: 1N4002, Diode_THT:D_DO-41_SOD81_P10.16mm_Horizontal, symbol Diode:1N4002
- removed Q2, Q3: SQJQ466E, Package_TO_SOT_SMD:LFPAK88, symbol Transistor_FET:SQJQ466E
- removed Q4: IRFR210PBF, Package_TO_SOT_SMD:TO-252-3_TabPin2, symbol Device:Q_NMOS_Depletion_GDS
- removed R11: 100R, Resistor_SMD:R_1206_3216Metric_Pad1.30x1.75mm_HandSolder, symbol PCM_Elektuur:R
- removed R12: 95.3k, Resistor_SMD:R_1206_3216Metric_Pad1.30x1.75mm_HandSolder, symbol PCM_Elektuur:R
- removed R13: 13.7k, Resistor_SMD:R_1206_3216Metric_Pad1.30x1.75mm_HandSolder, symbol PCM_Elektuur:R
- removed R14: 54.9k, Resistor_SMD:R_1206_3216Metric_Pad1.30x1.75mm_HandSolder, symbol PCM_Elektuur:R
- removed R15: 0.004R, Resistor_SMD:R_Shunt_Vishay_WSR2_WSR3_KelvinConnection, symbol PCM_Elektuur:R
- removed R3: 10k, Resistor_SMD:R_1206_3216Metric_Pad1.30x1.75mm_HandSolder, symbol PCM_Elektuur:R
- removed R5: 100k, Resistor_SMD:R_1206_3216Metric_Pad1.30x1.75mm_HandSolder, symbol PCM_Elektuur:R
- removed R6: 3.48K, Resistor_SMD:R_1206_3216Metric_Pad1.30x1.75mm_HandSolder, symbol PCM_Elektuur:R
- removed U1: LM74800QDRRRQ1, LM74800QDRRRQ1:IC_LM74800QDRRRQ1, symbol LM74800QDRRRQ1:LM74800QDRRRQ1
- removed U3: LM5069MM-2_NOPB, LM5069MM-2_NOPB:SOP50P490X110-10N, symbol LM5069MM-2_NOPB:LM5069MM-2_NOPB
Connections:
- net GND: no longer H1.1
- new net GNDS: H1.1
- no-connect marks 2 -> 0
Other:
- added sheet Stage1 (Stage1.kicad_sch)
- added sheet Stage2 (Stage2.kicad_sch)
- moved on the sheet: H1, H6, H7, H8

Commit message: new layout
Other:
- sheet Stage1 ports: added SYSOUT; removed OUT
Changed lines of the file:
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@@
 			)
 		)
-		(pin "OUT" output
+		(pin "SYSOUT" output
 			(at 86.36 72.39 0)
 			(effects

Commit message: smal changes
Connections:
- net GND is gone; now on net GNDS: H8.1
Changed lines of the file:
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@@
 	)
 	(symbol
-		(lib_id "power:GND")
+		(lib_id "power:GNDS")
 		(at 68.58 185.42 0)
 		(unit 1)
@@
 		(dnp no)
 		(fields_autoplaced yes)
-		(property "Reference" "#PWR020"
+		(property "Reference" "#PWR024"
 			(at 68.58 191.77 0)
 			(effects
@@
 			)
 		)
-		(property "Value" "GND"
+		(property "Value" "GNDS"
 			(at 68.58 190.5 0)
 			(effects
@@
 			)
 		)
-		(property "Description" "Power symbol creates a global label with name \"GND\" , ground"
+		(property "Description" "Power symbol creates a global label with name \"GNDS\" , signal ground"
 			(at 68.58 185.42 0)
 			(effects
@@
 			(project "OverVoltageProtection"
 				(path "/3ab01156-4af1-4058-a55c-fa6294991d75"
-					(reference "#PWR020")
+					(reference "#PWR024")
 					(unit 1)
 				)
