File: Stage2.kicad_sch (KiCad schematic)
At the start: 15 parts, among them Q2 SQJQ480E, U3 LM5069MM-2_NOPB

Commit message: new layout
Parts:
- removed D3: BAV20, Diode_THT:D_DO-35_SOD27_P7.62mm_Horizontal, symbol Diode:BAV20
- added D5: BAS20, Package_TO_SOT_SMD:SOT-23, symbol Diode:BAS20
- D7: footprint Diode_THT:D_DO-35_SOD27_P7.62mm_Horizontal -> Diode_SMD:D_SOD-123
Connections:
- net GND2: now also D5.1 (A)
- net GNDS: now also D5.3 (K)
Changed lines of the file:
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@@
 	)
 	(symbol
-		(lib_id "Diode:BAV20")
+		(lib_id "Diode:BAS20")
 		(at 175.26 121.92 180)
 		(unit 1)
@@
 		(dnp no)
 		(fields_autoplaced yes)
-		(property "Reference" "D3"
+		(property "Reference" "D5"
 			(at 175.26 115.57 0)
 			(effects
@@
 			)
 		)
-		(property "Value" "BAV20"
+		(property "Value" "BAS20"
 			(at 175.26 118.11 0)
 			(effects
@@
 			)
 		)
-		(property "Footprint" "Diode_THT:D_DO-35_SOD27_P7.62mm_Horizontal"
+		(property "Footprint" "Package_TO_SOT_SMD:SOT-23"
 			(at 175.26 117.475 0)
 			(effects
@@
 			)
 		)
-		(property "Datasheet" "http://www.vishay.com/docs/85543/bav17.pdf"
+		(property "Datasheet" "https://www.diodes.com/assets/Datasheets/Ds12004.pdf"
 			(at 175.26 121.92 0)
 			(effects
@@
 			)
 		)
-		(property "Description" "150V 0.25A Small Signal Switching Diode, High Voltage, DO-35"
+		(property "Description" "200V, 0.4A, High-speed Switching Diode, SOT-23"
 			(at 175.26 121.92 0)
 			(effects
@@
 			)
 		)
-		(property "Sim.Device" "D"
-			(at 175.26 121.92 0)
-			(effects
-				(font
-					(size 1.27 1.27)
-				)
-				(hide yes)
-			)
-		)
-		(property "Sim.Pins" "1=K 2=A"
-			(at 175.26 121.92 0)
-			(effects
-				(font
-					(size 1.27 1.27)
-				)
-				(hide yes)
-			)
-		)
-		(pin "1"
+		(pin "1"
+		)
+		(pin "3"
 		)
 		(pin "2"
 		)
 		(instances
-			(project "OverVoltageProtection"
-				(path "/3ab01156-4af1-4058-a55c-fa6294991d75/a98a8b2a-0085-4339-92cf-38a8f9617165"
-					(reference "D3")
+			(project ""
+				(path "/3ab01156-4af1-4058-a55c-fa6294991d75/a98a8b2a-0085-4339-92cf-38a8f9617165"
+					(reference "D5")
 					(unit 1)
 				)
@@
 			)
 		)
-		(property "Footprint" "Diode_THT:D_DO-35_SOD27_P7.62mm_Horizontal"
+		(property "Footprint" "Diode_SMD:D_SOD-123"
 			(at 165.735 106.68 0)
 			(effects

Commit message: smal changes
Connections:
- net GNDS is gone; now on net GND2: C13.2 (-), C17.2 (-), C18.2 (-), D5.3 (K), NT2.1
Other:
- moved on the sheet: NT2
Changed lines of the file:
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@@
+	)
+	(junction
+		(at 95.25 110.49)
+		(diameter 0)
+		(color 0 0 0 0)
+	)
+	(junction
+		(at 86.36 110.49)
+		(diameter 0)
+		(color 0 0 0 0)
 	)
 	(junction
@@
 	(wire
 		(pts
+			(xy 86.36 111.76) (xy 86.36 110.49)
+		)
+		(stroke
+			(width 0)
+			(type default)
+		)
+	)
+	(wire
+		(pts
 			(xy 185.42 77.47) (xy 198.12 77.47)
 		)
@@
 	(wire
 		(pts
-			(xy 82.55 110.49) (xy 87.63 110.49)
+			(xy 86.36 111.76) (xy 87.63 111.76)
 		)
 		(stroke
@@
 	(wire
 		(pts
+			(xy 86.36 110.49) (xy 95.25 110.49)
+		)
+		(stroke
+			(width 0)
+			(type default)
+		)
+	)
+	(wire
+		(pts
 			(xy 204.47 87.63) (xy 198.12 87.63)
 		)
@@
 	(wire
 		(pts
+			(xy 95.25 111.76) (xy 95.25 110.49)
+		)
+		(stroke
+			(width 0)
+			(type default)
+		)
+	)
+	(wire
+		(pts
 			(xy 170.18 102.87) (xy 170.18 99.06)
 		)
@@
 	(wire
 		(pts
-			(xy 92.71 110.49) (xy 97.79 110.49)
+			(xy 92.71 111.76) (xy 95.25 111.76)
 		)
 		(stroke
@@
 		(pts
 			(xy 97.79 91.44) (xy 102.87 91.44)
+		)
+		(stroke
+			(width 0)
+			(type default)
+		)
+	)
+	(wire
+		(pts
+			(xy 86.36 110.49) (xy 82.55 110.49)
+		)
+		(stroke
+			(width 0)
+			(type default)
+		)
+	)
+	(wire
+		(pts
+			(xy 95.25 110.49) (xy 97.79 110.49)
 		)
 		(stroke
@@
 	(symbol
 		(lib_id "Device:NetTie_2")
-		(at 90.17 110.49 0)
+		(at 90.17 111.76 0)
 		(unit 1)
 		(exclude_from_sim no)
@@
 		(dnp no)
 		(property "Reference" "NT2"
-			(at 90.17 112.268 0)
+			(at 90.17 113.538 0)
 			(effects
 				(font
@@
 		)
 		(property "Value" "NetTie_2"
-			(at 90.17 114.808 0)
+			(at 90.17 116.078 0)
 			(effects
 				(font
@@
 		)
 		(property "Footprint" ""
-			(at 90.17 110.49 0)
+			(at 90.17 111.76 0)
 			(effects
 				(font
@@
 		)
 		(property "Datasheet" "~"
-			(at 90.17 110.49 0)
+			(at 90.17 111.76 0)
 			(effects
 				(font
@@
 		)
 		(property "Description" "Net tie, 2 pins"
-			(at 90.17 110.49 0)
-			(effects
-				(font
+			(at 90.17 111.76 0)
+			(effects
+				(font

Commit message: fixed HW bug ?
Parts:
- removed Q2: SQJQ480E, Package_TO_SOT_SMD:LFPAK88, symbol Transistor_FET:SQJQ480E
- added Q9: SQJQ466E-T1_GE3, Package_TO_SOT_SMD:LFPAK88, symbol Transistor_FET:SQJQ480E
Connections:
- net GND2: no longer C13.2 (-), C17.2 (-), C18.2 (-), D5.3 (K), NT2.1
- net OUT: now also Q9.2 (S), Q9.3 (S), Q9.4 (S)
- net SENSE: now also Q9.5 (D)
- net at D7.1 (K), U3.10 (GATE): now also Q9.1 (G)
- new net GNDS: C13.2 (-), C17.2 (-), C18.2 (-), D5.3 (K), NT2.1
Other:
- moved on the sheet: NT2
Changed lines of the file:
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@@
-	)
-	(junction
-		(at 95.25 110.49)
-		(diameter 0)
-		(color 0 0 0 0)
-	)
-	(junction
-		(at 86.36 110.49)
-		(diameter 0)
-		(color 0 0 0 0)
 	)
 	(junction
@@
 	(wire
 		(pts
-			(xy 86.36 111.76) (xy 86.36 110.49)
-		)
-		(stroke
-			(width 0)
-			(type default)
-		)
-	)
-	(wire
-		(pts
 			(xy 185.42 77.47) (xy 198.12 77.47)
 		)
@@
 	(wire
 		(pts
-			(xy 86.36 111.76) (xy 87.63 111.76)
-		)
-		(stroke
-			(width 0)
-			(type default)
-		)
-	)
-	(wire
-		(pts
 			(xy 170.18 99.06) (xy 170.18 85.09)
 		)
@@
 	(wire
 		(pts
-			(xy 86.36 110.49) (xy 95.25 110.49)
-		)
-		(stroke
-			(width 0)
-			(type default)
-		)
-	)
-	(wire
-		(pts
 			(xy 204.47 87.63) (xy 198.12 87.63)
 		)
@@
 	(wire
 		(pts
-			(xy 95.25 111.76) (xy 95.25 110.49)
-		)
-		(stroke
-			(width 0)
-			(type default)
-		)
-	)
-	(wire
-		(pts
 			(xy 170.18 102.87) (xy 170.18 99.06)
 		)
@@
 	(wire
 		(pts
-			(xy 92.71 111.76) (xy 95.25 111.76)
+			(xy 92.71 110.49) (xy 97.79 110.49)
 		)
 		(stroke
@@
 	(wire
 		(pts
-			(xy 86.36 110.49) (xy 82.55 110.49)
-		)
-		(stroke
-			(width 0)
-			(type default)
-		)
-	)
-	(wire
-		(pts
-			(xy 95.25 110.49) (xy 97.79 110.49)
+			(xy 82.55 110.49) (xy 87.63 110.49)
 		)
 		(stroke
@@
 			)
 			(justify right)
-		)
-	)
-	(symbol
-		(lib_id "Transistor_FET:SQJQ480E")
-		(at 170.18 80.01 90)
-		(unit 1)
-		(exclude_from_sim no)
-		(in_bom yes)
-		(on_board yes)
-		(dnp no)
-		(fields_autoplaced yes)
-		(property "Reference" "Q2"
-			(at 170.18 71.12 90)
-			(effects
-				(font
-					(size 1.27 1.27)
-				)
-			)
-		)
-		(property "Value" "SQJQ480E"
-			(at 170.18 73.66 90)
-			(effects
-				(font
-					(size 1.27 1.27)
-				)
-			)
-		)
-		(property "Footprint" "Package_TO_SOT_SMD:LFPAK88"
-			(at 173.99 74.93 0)
-			(effects
-				(font
-					(size 1.27 1.27)
-				)
-				(justify left)
-				(hide yes)
-			)
-		)
-		(property "Datasheet" "https://www.vishay.com/docs/76718/sqjq480e.pdf"
-			(at 176.53 74.93 0)
-			(effects
-				(font
-					(size 1.27 1.27)
-				)
-				(justify left)
-				(hide yes)
-			)
-		)
-		(property "Description" "150A Id, 80V Vds, N-Channel TrenchFET MOSFET, 3mOhm Ron, 21nC Qqd, -55 to 175 °C, LFPAK88"
-			(at 170.18 80.01 0)
-			(effects
-				(font
-					(size 1.27 1.27)
-				)
-				(hide yes)
-			)
-		)
-		(pin "3"
-		)
-		(pin "2"
-		)
-		(pin "5"
-		)
-		(pin "4"
-		)
-		(pin "1"
-		)
-		(instances
-			(project "OverVoltageProtection"
-				(path "/3ab01156-4af1-4058-a55c-fa6294991d75/a98a8b2a-0085-4339-92cf-38a8f9617165"
-					(reference "Q2")
-					(unit 1)
-				)
-			)
 		)
 	)
@@
 	(symbol
 		(lib_id "Device:NetTie_2")
-		(at 90.17 111.76 0)
+		(at 90.17 110.49 0)
 		(unit 1)
 		(exclude_from_sim no)
@@
 		(dnp no)
 		(property "Reference" "NT2"
-			(at 90.17 113.538 0)
+			(at 90.17 112.268 0)
 			(effects
 				(font
@@
 		)
 		(property "Value" "NetTie_2"
-			(at 90.17 116.078 0)
+			(at 90.17 114.808 0)
 			(effects
 				(font
@@
 		)
 		(property "Footprint" ""
-			(at 90.17 111.76 0)
+			(at 90.17 110.49 0)
 			(effects
 				(font
@@
 		)
 		(property "Datasheet" "~"
-			(at 90.17 111.76 0)
+			(at 90.17 110.49 0)
 			(effects
 				(font
@@
 		)
 		(property "Description" "Net tie, 2 pins"
-			(at 90.17 111.76 0)
+			(at 90.17 110.49 0)
 			(effects
 				(font
@@
 					(unit 1)
 				)
+			)
+		)
+	)
+	(symbol
+		(lib_id "Transistor_FET:SQJQ480E")
+		(at 170.18 80.01 90)
+		(unit 1)
+		(exclude_from_sim no)
+		(in_bom yes)
+		(on_board yes)
+		(dnp no)
+		(property "Reference" "Q9"
+			(at 170.18 71.12 90)
+			(effects
+				(font
+					(size 1.27 1.27)
+				)
+			)
+		)
+		(property "Value" "SQJQ466E-T1_GE3"
+			(at 170.18 73.66 90)
+			(effects
+				(font
+					(size 1.27 1.27)
+				)
+			)
+		)
+		(property "Footprint" "Package_TO_SOT_SMD:LFPAK88"
+			(at 173.99 74.93 0)
+			(effects
+				(font
+					(size 1.27 1.27)
+				)
+				(justify left)
+				(hide yes)
+			)
+		)
+		(property "Datasheet" "https://www.vishay.com/docs/76718/sqjq480e.pdf"
+			(at 176.53 74.93 0)
+			(effects
+				(font
+					(size 1.27 1.27)
+				)
+				(justify left)
+				(hide yes)
+			)
+		)
+		(property "Description" "150A Id, 80V Vds, N-Channel TrenchFET MOSFET, 3mOhm Ron, 21nC Qqd, -55 to 175 °C, LFPAK88"
+			(at 170.18 80.01 0)
+			(effects
+				(font
+					(size 1.27 1.27)
+				)
+				(hide yes)
+			)
+		)
+		(pin "3"
+		)
+		(pin "2"
+		)
+		(pin "5"
+		)
+		(pin "4"
+		)
+		(pin "1"
+		)
+		(instances
+			(project "OverVoltageProtection"
+				(path "/3ab01156-4af1-4058-a55c-fa6294991d75/a98a8b2a-0085-4339-92cf-38a8f9617165"
+					(reference "Q9")
+					(unit 1)
+				)

Commit message: reworked schematics
Parts:
- C15: value 1000pF -> 1nF
- R12, R13, R14: footprint Resistor_SMD:R_1206_3216Metric_Pad1.30x1.75mm_HandSolder -> Resistor_SMD:R_1206_3216Metric
Changed lines of the file:
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@@
 			)
 		)
-		(property "Footprint" "Resistor_SMD:R_1206_3216Metric_Pad1.30x1.75mm_HandSolder"
+		(property "Footprint" "Resistor_SMD:R_1206_3216Metric"
 			(at 111.76 116.84 0)
 			(effects
@@
 			)
 		)
-		(property "Footprint" "Resistor_SMD:R_1206_3216Metric_Pad1.30x1.75mm_HandSolder"
+		(property "Footprint" "Resistor_SMD:R_1206_3216Metric"
 			(at 97.79 96.52 0)
 			(effects
@@
 			)
 		)
-		(property "Footprint" "Resistor_SMD:R_1206_3216Metric_Pad1.30x1.75mm_HandSolder"
+		(property "Footprint" "Resistor_SMD:R_1206_3216Metric"
 			(at 97.79 86.36 0)
 			(effects
@@
 			)
 		)
-		(property "Value" "1000pF"
+		(property "Value" "1nF"
 			(at 115.57 92.7099 0)
 			(effects

Commit message: updated layout
Parts:
- NT2: footprint (none) -> NetTie:NetTie-2_SMD_Pad0.5mm
Changed lines of the file:
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@@
 			)
 		)
-		(property "Footprint" ""
+		(property "Footprint" "NetTie:NetTie-2_SMD_Pad0.5mm"
 			(at 90.17 110.49 0)
 			(effects
